File: hardware/kicad_project/TiltTrack.kicad_sch (KiCad schematic)
At the start: 2 parts, among them J1 ESP32_DEVKIT_HEADER, J2 MPU6500_HEADER

Commit message: Updated Schematic
Parts:
- added J3: TOUCH_SENSOR_HEADER, symbol Connector:Conn_01x05_Pin
Connections:
- net +3V3: now also J3.4 (Pin_4)
- net GND: now also J3.1 (Pin_1), J3.3 (Pin_3)
- net TOUCH_OUT: now also J3.2 (Pin_2)
- no-connect marks 0 -> 29
